Commit message: checkpoint after generating obstacle swerving simulation

File: src/robotino_description/urdf/robotino_platform.urdf.xacro (robot description, xacro)
@@ -1,10 +1,10 @@
 <?xml version="1.0"?>
 <robot name="robotino" xmlns:xacro="http://wiki.ros.org/xacro">
-    <xacro:include filename="$(find robotino_description)/urdf/robotino_body.urdf.xacro"/>
-    <xacro:include filename="$(find robotino_description)/urdf/robotino_parts.urdf.xacro"/>
-    <xacro:robotino_body/>
+    <xacro:include filename="$(find robotino_description)/urdf/robotino_body.urdf.xacro" />
+    <xacro:include filename="$(find robotino_description)/urdf/robotino_parts.urdf.xacro" />
+    <xacro:robotino_body />
     <!-- add platform -->
-    <platform name="platform" parent="base_link">
-        <origin xyz="0.0 0.0 0.13" rpy="0 0 0"/>
-    </platform>
+    <xacro:platform name="platform" parent="base_link">
+      <origin xyz="0.0 0.0 0.13" rpy="0 0 0" />
+    </xacro:platform>
 </robot>
